File: pcb-power/pcb-power.kicad_pcb (KiCad board)
At the start: 2 copper layers, 152.4 x 101.6 mm, 91 parts, among them Q1 IPN70R1K5CE, U1 UC3845, U2 7809, U3 7909, X1 PH, X2 N, X3 G, X4 +9V, X5 -9V, X6 H1, X7 H2, X8 +400V, X9 -400V

Commit message: Before second re-route
Parts:
- removed SYM1: SYM_Flash_Small, Symbol:Symbol_HighVoltage_Type2_CopperTop_VerySmall
Other:
- board text added: "DANGER! HIGH VOLTAGE in excess of ±400V with lethal current in all areas. Contact may KILL. System may retain charge."
- board text removed: "DANGER! HIGH VOLTAGE in excess of ±400V with lethal current. Contact may result in serious injury or death. System may retain charge."

Commit message: Cleaned up
Parts:
- renumbered X4 to X12, X5 to X13, X8 to X14, X9 to X15, X2 to XJ2.2, X3 to XJ2.3, X6 to XR1, X1 to XSW1, X7 to XV1.14
Routing:
- net /VSW: track 68.0 -> 66.6 mm

Commit message: Version sent to fab
Parts:
- added R16: 750, Resistor_THT:R_Axial_DIN0207_L6.3mm_D2.5mm_P10.16mm_Horizontal, F.Cu at (36.2, 66.7)
- added R17: 120, Resistor_THT:R_Axial_DIN0207_L6.3mm_D2.5mm_P10.16mm_Horizontal, F.Cu at (33.0, 66.7)
- C13: value 220p/500V -> 100p/500V; footprint Capacitor_THT:C_Disc_D7.5mm_W5.0mm_P10.00mm -> Capacitor_THT:C_Disc_D7.0mm_W2.5mm_P5.00mm
- D8, D9: value 1N4004 -> 1N4007
- RV1: footprint Potentiometer_THT:Potentiometer_Bourns_3339P_Vertical -> mini-audioscope:stock_pot
- U1: value UC3845 -> UC3843
- U3: value 7909 -> LM337
- X12, X13, X14, X15, XJ2.2, XJ2.3, XR1, XSW1, XT1.0, XT1.1, XT1.2, XT1.3, XT1.4, XT1.6, XT1.8, XT1.9, XV1.14: footprint Connector_Pin:Pin_D0.7mm_L6.5mm_W1.8mm_FlatFork -> Connector_Pin:Pin_D1.1mm_L8.5mm_W2.5mm_FlatFork
- moved C13 6.43 mm to (108.0, 100.2)
- moved XT1.9 5.08 mm to (86.4, 33.0)
- moved XT1.1 3.81 mm to (71.1, 33.0)
- moved TP4 3.42 mm to (104.1, 75.6)
- moved R10 2.62 mm to (108.0, 79.4)
- moved XT1.2 2.54 mm to (99.1, 33.0)
- moved XT1.6 2.54 mm to (94.0, 33.0)
- moved XT1.3 2.54 mm to (78.7, 33.0)
- moved RV1 2.09 mm to (67.1, 109.7)
- moved XT1.0 1.27 mm to (63.5, 33.0)
Connections:
- U3 pad 1: GND -> Net-(R16-Pad2)
Routing:
- net Net-(R16-Pad2): track 0.00 -> 10.9 mm
- net Net-(C24-Pad2): track 18.0 -> 28.5 mm
- net /NEUT: track 71.4 -> 80.4 mm
- net Net-(C13-Pad1): track 23.1 -> 18.4 mm
- net /LINE_NTC: track 20.8 -> 24.5 mm
- net Net-(C17-Pad1): track 56.7 -> 60.1 mm
- net Net-(D5-Pad2): track 41.9 -> 45.1 mm
- net /SNUB: track 5.02 -> 3.17 mm
- net Net-(C1-Pad1): track 34.6 -> 32.7 mm
- net /MULT4_250: track 27.4 -> 29.1 mm
- net /MULT2_250: track 34.8 -> 36.4 mm
- net Net-(C2-Pad1): track 32.0 -> 33.4 mm
- net /MULT1_400: track 17.4 -> 18.8 mm
- net Net-(R3-Pad2): track 7.32 -> 8.67 mm
- net Net-(C21-Pad2): track 26.2 -> 27.1 mm
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Other:
- outline, holes or cut-outs redrawn
- net class 250: clearance 1.25 -> 1.27; trace_width 0.25 -> 0.508; via_dia 0.8 -> 0.8128; via_drill 0.4 -> 0.4064
- net class 400: clearance 2.5 -> 2.54; trace_width 0.5 -> 0.508; via_dia 0.8 -> 0.8128; via_drill 0.4 -> 0.4064
- net class Default: clearance 0.2 -> 0.254; trace_width 0.25 -> 0.508; via_dia 0.8 -> 0.8128; via_drill 0.4 -> 0.4064
- net class Mains: clearance 1.25 -> 1.27; trace_width 0.25 -> 0.508; via_dia 0.8 -> 0.8128; via_drill 0.4 -> 0.4064
- rule trace_clearance: 0.2 -> 0.254
- board text removed: "[HV!]"
