File: mini-audioscope.kicad_pcb (KiCad board)
At the start: 2 copper layers, 0 parts

Commit message: Commit before re-routing
Parts:
- added C1: DNP, Capacitor_THT:C_Disc_D4.7mm_W2.5mm_P5.00mm, F.Cu at (47.0, 96.5)
- added C26: DNP, Capacitor_THT:C_Disc_D4.7mm_W2.5mm_P5.00mm, F.Cu at (88.3, 69.2)
- added C27: 100n, Capacitor_THT:C_Disc_D4.7mm_W2.5mm_P5.00mm, F.Cu at (76.8, 99.7)
- added C28: 330n, Capacitor_THT:C_Rect_L9.0mm_W4.2mm_P7.50mm_MKT, F.Cu at (57.1, 113.0)
- added C29: 330n, Capacitor_THT:C_Rect_L9.0mm_W4.2mm_P7.50mm_MKT, F.Cu at (52.7, 113.0)
- added C30: 47p, Capacitor_THT:C_Disc_D4.7mm_W2.5mm_P5.00mm, F.Cu at (72.4, 102.9)
- added C31: 22p, Capacitor_THT:C_Disc_D3.8mm_W2.6mm_P2.50mm, F.Cu at (88.3, 111.8)
- added C32: 3u3, Capacitor_THT:CP_Radial_D10.0mm_P2.50mm_P5.00mm, F.Cu at (106.7, 109.2)
- added C33: 10n, Capacitor_THT:C_Disc_D4.7mm_W2.5mm_P5.00mm, F.Cu at (105.4, 68.6)
- added C34: 100n, Capacitor_THT:C_Disc_D4.7mm_W2.5mm_P5.00mm, F.Cu at (105.4, 94.6)
- added C35: 100n, Capacitor_THT:C_Disc_D4.7mm_W2.5mm_P5.00mm, F.Cu at (118.1, 44.5)
- added C36: 47u, Capacitor_THT:CP_Radial_D6.3mm_P2.50mm, F.Cu at (107.3, 78.1)
- added C37: 10n, Capacitor_THT:C_Disc_D4.7mm_W2.5mm_P5.00mm, F.Cu at (106.0, 82.5)
- added C38: 470n, Capacitor_THT:C_Rect_L9.0mm_W5.1mm_P7.50mm_MKT, F.Cu at (97.8, 54.6)
- added C39: 470n, Capacitor_THT:C_Disc_D4.7mm_W2.5mm_P5.00mm, F.Cu at (88.4, 84.3)
- added D1: 1N4007, Diode_THT:D_DO-41_SOD81_P10.16mm_Horizontal, F.Cu at (127.0, 69.2)
- added D19: 1N4007, Diode_THT:D_DO-41_SOD81_P10.16mm_Horizontal, F.Cu at (62.2, 67.9)
- added D2: 1N4007, Diode_THT:D_DO-41_SOD81_P10.16mm_Horizontal, F.Cu at (123.8, 69.2)
- added D20: 1N4007, Diode_THT:D_DO-41_SOD81_P10.16mm_Horizontal, F.Cu at (68.6, 67.9)
- added D21: 1N4148, Diode_THT:D_DO-35_SOD27_P7.62mm_Horizontal, F.Cu at (99.1, 47.0)
- added D22: 1N4148, Diode_THT:D_DO-35_SOD27_P7.62mm_Horizontal, F.Cu at (94.6, 62.2)
- added D3: 1N4007, Diode_THT:D_DO-41_SOD81_P10.16mm_Horizontal, F.Cu at (158.1, 47.6)
- added D4: 1N4007, Diode_THT:D_DO-41_SOD81_P10.16mm_Horizontal, F.Cu at (43.8, 67.9)
- added D5: 1N4007, Diode_THT:D_DO-41_SOD81_P10.16mm_Horizontal, F.Cu at (50.2, 67.9)
- added H1: GND, MountingHole:MountingHole_4.3mm_M4_Pad_Via, F.Cu at (33.0, 33.0)
- added H2: GND, MountingHole:MountingHole_4.3mm_M4_Pad_Via, F.Cu at (33.0, 119.4)
- added H3: GND, MountingHole:MountingHole_4.3mm_M4_Pad_Via, F.Cu at (170.2, 119.4)
- added H4: GND, MountingHole:MountingHole_4.3mm_M4_Pad_Via, F.Cu at (170.2, 33.0)
- added NE1: A9A, Capacitor_THT:C_Radial_D8.0mm_H11.5mm_P3.50mm, F.Cu at (144.8, 42.5)
- added NE2: A9A, Capacitor_THT:C_Radial_D8.0mm_H11.5mm_P3.50mm, F.Cu at (153.7, 42.5)
- added NE5: A9A, Capacitor_THT:C_Radial_D8.0mm_H11.5mm_P3.50mm, F.Cu at (54.0, 84.5)
- added Q1: 2N3906, Package_TO_SOT_THT:TO-92_Inline, F.Cu at (123.8, 65.4)
- added Q11: 2N5551, Package_TO_SOT_THT:TO-92_Inline, F.Cu at (77.5, 71.1)
- added Q12: 2N4401, Package_TO_SOT_THT:TO-92_Inline, F.Cu at (80.9, 57.8)
- added Q13: ZTX458, Package_TO_SOT_THT:TO-5-3, F.Cu at (63.0, 64.1)
- added Q14: ZTX458, Package_TO_SOT_THT:TO-5-3, F.Cu at (72.9, 64.1)
- added Q15: 2N4401, Package_TO_SOT_THT:TO-92_Inline, F.Cu at (86.0, 57.8)
- added Q16: 2N5551, Package_TO_SOT_THT:TO-92_Inline, F.Cu at (77.5, 76.2)
- added Q17: 2N3906, Package_TO_SOT_THT:TO-92_Inline, F.Cu at (94.0, 108.6)
- added Q18: 2N3904, Package_TO_SOT_THT:TO-92_Inline, F.Cu at (87.9, 80.8)
- added Q19: 2N3906, Package_TO_SOT_THT:TO-92_Inline, F.Cu at (115.6, 99.7)
- added Q2: ZTX558, Package_TO_SOT_THT:TO-5-3, F.Cu at (134.0, 79.4)
- added Q20: 2N3904, Package_TO_SOT_THT:TO-92_Inline, F.Cu at (119.4, 108.0)
- added Q21: 2N3906, Package_TO_SOT_THT:TO-92_Inline, F.Cu at (109.9, 71.8)
- added Q22: 2N3906, Package_TO_SOT_THT:TO-92_Inline, F.Cu at (106.7, 66.0)
- added Q23: 2N3904, Package_TO_SOT_THT:TO-92_Inline, F.Cu at (103.5, 52.1)
- added Q3: ZTX558, Package_TO_SOT_THT:TO-5-3, F.Cu at (134.0, 69.2)
- added Q4: 2N5551, Package_TO_SOT_THT:TO-92_Inline, F.Cu at (41.9, 83.8)
- added Q5: 2N4401, Package_TO_SOT_THT:TO-92_Inline, F.Cu at (41.3, 102.2)
- added Q6: ZTX458, Package_TO_SOT_THT:TO-5-3, F.Cu at (43.2, 64.1)
- added Q7: ZTX458, Package_TO_SOT_THT:TO-5-3, F.Cu at (53.1, 64.1)
- added Q8: 2N4401, Package_TO_SOT_THT:TO-92_Inline, F.Cu at (46.4, 102.2)
- added Q9: 2N5551, Package_TO_SOT_THT:TO-92_Inline, F.Cu at (47.0, 83.8)
- added R1: 100k, Resistor_THT:R_Axial_DIN0207_L6.3mm_D2.5mm_P10.16mm_Horizontal, F.Cu at (120.0, 92.7)
- added R10: 20k, Resistor_THT:R_Axial_DIN0207_L6.3mm_D2.5mm_P10.16mm_Horizontal, F.Cu at (120.7, 79.4)
- added R11: 220k/HW, Resistor_THT:R_Axial_DIN0309_L9.0mm_D3.2mm_P12.70mm_Horizontal, F.Cu at (141.0, 51.4)
- added R12: 100k/HW, Resistor_THT:R_Axial_DIN0309_L9.0mm_D3.2mm_P12.70mm_Horizontal, F.Cu at (149.2, 60.3)
- added R13: 10k, Resistor_THT:R_Axial_DIN0207_L6.3mm_D2.5mm_P10.16mm_Horizontal, F.Cu at (121.9, 42.5)
- added R14: 330k/HW, Resistor_THT:R_Axial_DIN0309_L9.0mm_D3.2mm_P12.70mm_Horizontal, F.Cu at (125.7, 41.9)
- added R15: 10k/HW, Resistor_THT:R_Axial_DIN0309_L9.0mm_D3.2mm_P12.70mm_Horizontal, F.Cu at (76.2, 40.0)
- added R16: 390k/HW, Resistor_THT:R_Axial_DIN0309_L9.0mm_D3.2mm_P12.70mm_Horizontal, F.Cu at (152.4, 75.6)
- added R17: 390k/HW, Resistor_THT:R_Axial_DIN0309_L9.0mm_D3.2mm_P12.70mm_Horizontal, F.Cu at (153.7, 60.3)
- added R18: 220k/HW, Resistor_THT:R_Axial_DIN0309_L9.0mm_D3.2mm_P12.70mm_Horizontal, F.Cu at (162.6, 82.5)
- added R19: 100k/HW, Resistor_THT:R_Axial_DIN0309_L9.0mm_D3.2mm_P12.70mm_Horizontal, F.Cu at (157.5, 85.1)
- added R20: 10k, Resistor_THT:R_Axial_DIN0207_L6.3mm_D2.5mm_P10.16mm_Horizontal, F.Cu at (69.8, 95.2)
- added R21: 10k, Resistor_THT:R_Axial_DIN0207_L6.3mm_D2.5mm_P10.16mm_Horizontal, F.Cu at (59.7, 98.4)
- added R22: 220k/HW, Resistor_THT:R_Axial_DIN0309_L9.0mm_D3.2mm_P12.70mm_Horizontal, F.Cu at (43.2, 39.4)
- added R23: 470, Resistor_THT:R_Axial_DIN0207_L6.3mm_D2.5mm_P10.16mm_Horizontal, F.Cu at (40.6, 67.9)
- added R24: 8k2, Resistor_THT:R_Axial_DIN0207_L6.3mm_D2.5mm_P10.16mm_Horizontal, F.Cu at (40.6, 105.4)
- added R25: 1k5, Resistor_THT:R_Axial_DIN0207_L6.3mm_D2.5mm_P10.16mm_Horizontal, F.Cu at (40.6, 86.4)
- added R26: DNP, Resistor_THT:R_Axial_DIN0207_L6.3mm_D2.5mm_P10.16mm_Horizontal, F.Cu at (43.8, 86.4)
- added R27: 10k, Resistor_THT:R_Axial_DIN0207_L6.3mm_D2.5mm_P10.16mm_Horizontal, F.Cu at (59.1, 78.1)
- added R28: 220k/HW, Resistor_THT:R_Axial_DIN0309_L9.0mm_D3.2mm_P12.70mm_Horizontal, F.Cu at (50.8, 39.4)
- added R29: 470, Resistor_THT:R_Axial_DIN0207_L6.3mm_D2.5mm_P10.16mm_Horizontal, F.Cu at (47.0, 67.9)
- added R3: 470k, Resistor_THT:R_Axial_DIN0207_L6.3mm_D2.5mm_P10.16mm_Horizontal, F.Cu at (117.5, 83.8)
- added R30: 8k2, Resistor_THT:R_Axial_DIN0207_L6.3mm_D2.5mm_P10.16mm_Horizontal, F.Cu at (59.7, 101.6)
- added R31: 10k/HW, Resistor_THT:R_Axial_DIN0309_L9.0mm_D3.2mm_P12.70mm_Horizontal, F.Cu at (47.0, 54.6)
- added R32: 10k/HW, Resistor_THT:R_Axial_DIN0309_L9.0mm_D3.2mm_P12.70mm_Horizontal, F.Cu at (54.6, 54.6)
- added R33: 10k, Resistor_THT:R_Axial_DIN0207_L6.3mm_D2.5mm_P10.16mm_Horizontal, F.Cu at (48.3, 105.4)
- added R34: 10k, Resistor_THT:R_Axial_DIN0207_L6.3mm_D2.5mm_P10.16mm_Horizontal, F.Cu at (45.1, 115.6)
- added R4: 1k, Resistor_THT:R_Axial_DIN0207_L6.3mm_D2.5mm_P10.16mm_Horizontal, F.Cu at (130.2, 87.0)
- added R46: 10k, Resistor_THT:R_Axial_DIN0207_L6.3mm_D2.5mm_P10.16mm_Horizontal, F.Cu at (83.8, 45.1)
- added R47: 10k, Resistor_THT:R_Axial_DIN0207_L6.3mm_D2.5mm_P10.16mm_Horizontal, F.Cu at (87.0, 55.2)
- added R48: 220k/HW, Resistor_THT:R_Axial_DIN0309_L9.0mm_D3.2mm_P12.70mm_Horizontal, F.Cu at (58.4, 39.4)
- added R49: 470, Resistor_THT:R_Axial_DIN0207_L6.3mm_D2.5mm_P10.16mm_Horizontal, F.Cu at (65.4, 67.9)
- added R5: 33k, Resistor_THT:R_Axial_DIN0207_L6.3mm_D2.5mm_P10.16mm_Horizontal, F.Cu at (111.1, 62.2)
- added R50: 8k2, Resistor_THT:R_Axial_DIN0207_L6.3mm_D2.5mm_P10.16mm_Horizontal, F.Cu at (77.5, 55.2)
- added R51: 1k5, Resistor_THT:R_Axial_DIN0207_L6.3mm_D2.5mm_P10.16mm_Horizontal, F.Cu at (80.6, 74.9)
- added R52: DNP, Resistor_THT:R_Axial_DIN0207_L6.3mm_D2.5mm_P10.16mm_Horizontal, F.Cu at (80.6, 71.8)
- added R53: 10k, Resistor_THT:R_Axial_DIN0207_L6.3mm_D2.5mm_P10.16mm_Horizontal, F.Cu at (74.3, 45.1)
- added R54: 220k/HW, Resistor_THT:R_Axial_DIN0309_L9.0mm_D3.2mm_P12.70mm_Horizontal, F.Cu at (66.0, 39.4)
- added R55: 470, Resistor_THT:R_Axial_DIN0207_L6.3mm_D2.5mm_P10.16mm_Horizontal, F.Cu at (71.8, 67.9)
- added R56: 8k2, Resistor_THT:R_Axial_DIN0207_L6.3mm_D2.5mm_P10.16mm_Horizontal, F.Cu at (80.6, 55.2)
- added R57: 10k/HW, Resistor_THT:R_Axial_DIN0309_L9.0mm_D3.2mm_P12.70mm_Horizontal, F.Cu at (62.2, 54.6)
- added R58: 10k/HW, Resistor_THT:R_Axial_DIN0309_L9.0mm_D3.2mm_P12.70mm_Horizontal, F.Cu at (69.8, 54.6)
- added R59: 10k, Resistor_THT:R_Axial_DIN0207_L6.3mm_D2.5mm_P10.16mm_Horizontal, F.Cu at (69.8, 85.7)
- added R6: 10k, Resistor_THT:R_Axial_DIN0207_L6.3mm_D2.5mm_P10.16mm_Horizontal, F.Cu at (130.2, 83.8)
- added R60: 10k, Resistor_THT:R_Axial_DIN0207_L6.3mm_D2.5mm_P10.16mm_Horizontal, F.Cu at (59.7, 82.5)
- added R61: 100k, Resistor_THT:R_Axial_DIN0207_L6.3mm_D2.5mm_P10.16mm_Horizontal, F.Cu at (61.6, 105.4)
- added R62: 100k, Resistor_THT:R_Axial_DIN0207_L6.3mm_D2.5mm_P10.16mm_Horizontal, F.Cu at (64.8, 105.4)
- added R64: 100k, Resistor_THT:R_Axial_DIN0207_L6.3mm_D2.5mm_P10.16mm_Horizontal, F.Cu at (67.9, 115.6)
- added R65: 1M, Resistor_THT:R_Axial_DIN0207_L6.3mm_D2.5mm_P10.16mm_Horizontal, F.Cu at (85.1, 105.4)
- added R66: 10k, Resistor_THT:R_Axial_DIN0207_L6.3mm_D2.5mm_P10.16mm_Horizontal, F.Cu at (81.9, 105.4)
- added R67: 27k, Resistor_THT:R_Axial_DIN0207_L6.3mm_D2.5mm_P10.16mm_Horizontal, F.Cu at (69.8, 88.9)
- added R68: 27k, Resistor_THT:R_Axial_DIN0207_L6.3mm_D2.5mm_P10.16mm_Horizontal, F.Cu at (59.7, 92.1)
- added R69: 4k7, Resistor_THT:R_Axial_DIN0207_L6.3mm_D2.5mm_P10.16mm_Horizontal, F.Cu at (88.3, 108.0)
- added R7: 180k, Resistor_THT:R_Axial_DIN0207_L6.3mm_D2.5mm_P10.16mm_Horizontal, F.Cu at (111.1, 65.4)
- added R70: 10k, Resistor_THT:R_Axial_DIN0207_L6.3mm_D2.5mm_P10.16mm_Horizontal, F.Cu at (85.1, 90.9)
- added R71: 4M7, Resistor_THT:R_Axial_DIN0207_L6.3mm_D2.5mm_P10.16mm_Horizontal, F.Cu at (91.4, 99.7)
- added R72: 10k, Resistor_THT:R_Axial_DIN0207_L6.3mm_D2.5mm_P10.16mm_Horizontal, F.Cu at (104.1, 91.4)
- added R73: 100k, Resistor_THT:R_Axial_DIN0207_L6.3mm_D2.5mm_P10.16mm_Horizontal, F.Cu at (80.6, 88.3)
- added R74: 10, Resistor_THT:R_Axial_DIN0207_L6.3mm_D2.5mm_P10.16mm_Horizontal, F.Cu at (97.8, 115.6)
- added R75: 100k, Resistor_THT:R_Axial_DIN0207_L6.3mm_D2.5mm_P10.16mm_Horizontal, F.Cu at (101.0, 105.4)
- added R76: 10k, Resistor_THT:R_Axial_DIN0207_L6.3mm_D2.5mm_P10.16mm_Horizontal, F.Cu at (108.6, 92.7)
- added R77: 22k, Resistor_THT:R_Axial_DIN0207_L6.3mm_D2.5mm_P10.16mm_Horizontal, F.Cu at (111.8, 102.9)
- added R78: 100k, Resistor_THT:R_Axial_DIN0207_L6.3mm_D2.5mm_P10.16mm_Horizontal, F.Cu at (83.8, 78.1)
- added R79: 100k, Resistor_THT:R_Axial_DIN0207_L6.3mm_D2.5mm_P10.16mm_Horizontal, F.Cu at (114.9, 105.4)
- added R8: 220k/HW, Resistor_THT:R_Axial_DIN0309_L9.0mm_D3.2mm_P12.70mm_Horizontal, F.Cu at (144.8, 79.4)
- added R80: 470, Resistor_THT:R_Axial_DIN0207_L6.3mm_D2.5mm_P10.16mm_Horizontal, F.Cu at (116.8, 79.4)
- added R81: 470, Resistor_THT:R_Axial_DIN0207_L6.3mm_D2.5mm_P10.16mm_Horizontal, F.Cu at (114.9, 83.8)
- added R82: 470, Resistor_THT:R_Axial_DIN0207_L6.3mm_D2.5mm_P10.16mm_Horizontal, F.Cu at (113.7, 79.4)
- added R83: 100, Resistor_THT:R_Axial_DIN0207_L6.3mm_D2.5mm_P10.16mm_Horizontal, F.Cu at (107.3, 55.9)
- added R84: 6k8, Resistor_THT:R_Axial_DIN0207_L6.3mm_D2.5mm_P10.16mm_Horizontal, F.Cu at (99.7, 50.2)
- added R85: 75k, Resistor_THT:R_Axial_DIN0207_L6.3mm_D2.5mm_P10.16mm_Horizontal, F.Cu at (94.0, 76.8)
- added R86: 10k, Resistor_THT:R_Axial_DIN0207_L6.3mm_D2.5mm_P10.16mm_Horizontal, F.Cu at (94.0, 44.5)
- added R87: 10k, Resistor_THT:R_Axial_DIN0207_L6.3mm_D2.5mm_P10.16mm_Horizontal, F.Cu at (104.1, 41.3)
- added R88: 10k, Resistor_THT:R_Axial_DIN0207_L6.3mm_D2.5mm_P10.16mm_Horizontal, F.Cu at (104.8, 59.1)
- added R89: 2k7, Resistor_THT:R_Axial_DIN0207_L6.3mm_D2.5mm_P10.16mm_Horizontal, F.Cu at (91.4, 59.1)
- added R9: 220k/HW, Resistor_THT:R_Axial_DIN0309_L9.0mm_D3.2mm_P12.70mm_Horizontal, F.Cu at (144.8, 51.4)
- added R90: 4M7, Resistor_THT:R_Axial_DIN0207_L6.3mm_D2.5mm_P10.16mm_Horizontal, F.Cu at (108.0, 41.3)
- added R91: 10k, Resistor_THT:R_Axial_DIN0207_L6.3mm_D2.5mm_P10.16mm_Horizontal, F.Cu at (107.3, 59.1)
- added RV1: 5k, Potentiometer_THT:Potentiometer_Bourns_3339P_Vertical, F.Cu at (134.6, 94.0)
- added RV2: 1M, Potentiometer_THT:Potentiometer_Bourns_3386P_Vertical, F.Cu at (132.1, 52.1)
- added RV3: 1M, Potentiometer_THT:Potentiometer_Bourns_3386P_Vertical, F.Cu at (153.7, 95.2)
- added RV4: 5k, Potentiometer_THT:Potentiometer_Bourns_3339P_Vertical, F.Cu at (52.7, 94.0)
- added RV5: 2k5, Potentiometer_THT:Potentiometer_Bourns_3339P_Vertical, F.Cu at (50.2, 99.7)
- added RV7: 5k, Potentiometer_THT:Potentiometer_Bourns_3339P_Vertical, F.Cu at (82.3, 68.6)
- added RV8: 2k5, Potentiometer_THT:Potentiometer_Bourns_3339P_Vertical, F.Cu at (74.9, 81.3)
- added RV9: 5k, Potentiometer_THT:Potentiometer_Bourns_3339P_Vertical, F.Cu at (79.4, 90.8)
- added TP1: V(A1), TestPoint:TestPoint_Loop_D2.60mm_Drill1.4mm_Beaded, F.Cu at (135.3, 57.8)
- added TP2: V(F), TestPoint:TestPoint_Loop_D2.60mm_Drill1.4mm_Beaded, F.Cu at (170.2, 44.5)
- added TP3: V(G), TestPoint:TestPoint_Loop_D2.60mm_Drill1.4mm_Beaded, F.Cu at (158.8, 64.8)
- added TP4: V(K), TestPoint:TestPoint_Loop_D2.60mm_Drill1.4mm_Beaded, F.Cu at (162.6, 44.5)
- added TP5: INTEN, TestPoint:TestPoint_Loop_D2.60mm_Drill1.4mm_Beaded, F.Cu at (144.8, 83.8)
- added TP6: GND, TestPoint:TestPoint_Loop_D2.60mm_Drill1.4mm_Beaded, F.Cu at (151.1, 80.0)
- added U4: TL072, Package_DIP:DIP-8_W7.62mm_LongPads, F.Cu at (71.1, 106.0)
- added U5: LM311, Package_DIP:DIP-8_W7.62mm_LongPads, F.Cu at (94.6, 94.6)
- added U6: NE555P, Package_DIP:DIP-8_W7.62mm_LongPads, F.Cu at (94.6, 65.4)
- added U7: NE555P, Package_DIP:DIP-8_W7.62mm_LongPads, F.Cu at (94.6, 80.0)
- added U8: LM311, Package_DIP:DIP-8_W7.62mm_LongPads, F.Cu at (107.3, 45.1)
- added X1: SLOPE, Connector_Pin:Pin_D0.7mm_L6.5mm_W1.8mm_FlatFork, F.Cu at (113.0, 121.9)
- added X10: IW, Connector_Pin:Pin_D0.7mm_L6.5mm_W1.8mm_FlatFork, F.Cu at (127.0, 121.9)
- added X11: IB, Connector_Pin:Pin_D0.7mm_L6.5mm_W1.8mm_FlatFork, F.Cu at (132.1, 121.9)
- added X12: +9, Connector_Pin:Pin_D0.7mm_L6.5mm_W1.8mm_FlatFork, F.Cu at (30.5, 101.6)
- added X13: -9, Connector_Pin:Pin_D0.7mm_L6.5mm_W1.8mm_FlatFork, F.Cu at (30.5, 95.2)
- added X14: +400, Connector_Pin:Pin_D0.7mm_L6.5mm_W1.8mm_FlatFork, F.Cu at (74.9, 33.0)
- added X15: -400, Connector_Pin:Pin_D0.7mm_L6.5mm_W1.8mm_FlatFork, F.Cu at (171.4, 96.5)
- added X2: NORM, Connector_Pin:Pin_D0.7mm_L6.5mm_W1.8mm_FlatFork, F.Cu at (108.0, 121.9)
- added X3: L, Connector_Pin:Pin_D0.7mm_L6.5mm_W1.8mm_FlatFork, F.Cu at (57.1, 121.9)
- added X4: R, Connector_Pin:Pin_D0.7mm_L6.5mm_W1.8mm_FlatFork, F.Cu at (52.1, 121.9)
- added X5: G, Connector_Pin:Pin_D0.7mm_L6.5mm_W1.8mm_FlatFork, F.Cu at (47.0, 121.9)
- added X6: GO, Connector_Pin:Pin_D0.7mm_L6.5mm_W1.8mm_FlatFork, F.Cu at (74.9, 121.9)
- added X7: GI, Connector_Pin:Pin_D0.7mm_L6.5mm_W1.8mm_FlatFork, F.Cu at (80.0, 121.9)
- added X8: GG, Connector_Pin:Pin_D0.7mm_L6.5mm_W1.8mm_FlatFork, F.Cu at (85.1, 121.9)
- added X9: IT, Connector_Pin:Pin_D0.7mm_L6.5mm_W1.8mm_FlatFork, F.Cu at (121.9, 121.9)
- added XV1.10: V+, Connector_Pin:Pin_D0.7mm_L6.5mm_W1.8mm_FlatFork, F.Cu at (50.8, 33.0)
- added XV1.11: V-, Connector_Pin:Pin_D0.7mm_L6.5mm_W1.8mm_FlatFork, F.Cu at (45.7, 33.0)
- added XV1.2: K, Connector_Pin:Pin_D0.7mm_L6.5mm_W1.8mm_FlatFork, F.Cu at (154.9, 33.0)
- added XV1.3: G, Connector_Pin:Pin_D0.7mm_L6.5mm_W1.8mm_FlatFork, F.Cu at (148.6, 33.0)
- added XV1.4: A1, Connector_Pin:Pin_D0.7mm_L6.5mm_W1.8mm_FlatFork, F.Cu at (111.8, 33.0)
- added XV1.6: F, Connector_Pin:Pin_D0.7mm_L6.5mm_W1.8mm_FlatFork, F.Cu at (161.3, 33.0)
- added XV1.7: X-, Connector_Pin:Pin_D0.7mm_L6.5mm_W1.8mm_FlatFork, F.Cu at (63.5, 33.0)
- added XV1.8: X+, Connector_Pin:Pin_D0.7mm_L6.5mm_W1.8mm_FlatFork, F.Cu at (68.6, 33.0)
- added XV1.9: A2, Connector_Pin:Pin_D0.7mm_L6.5mm_W1.8mm_FlatFork, F.Cu at (104.1, 33.0)
Routing:
- net +9V: track 0.00 -> 415.4 mm, vias 0 -> 1
- net -9V: track 0.00 -> 291.0 mm, vias 0 -> 7
- net -400V: track 0.00 -> 108.7 mm, vias 0 -> 1
- net /K: track 0.00 -> 87.5 mm
- net /OUT: track 0.00 -> 85.0 mm
- net GND: track 0.00 -> 76.1 mm
- net /~NORM: track 0.00 -> 66.3 mm
- net Net-(D21-Pad2): track 0.00 -> 63.9 mm
- net /F: track 0.00 -> 51.3 mm
- net /INTEN_W: track 0.00 -> 49.4 mm
- net /~BLANK: track 0.00 -> 49.0 mm
- net +400V: track 0.00 -> 47.6 mm
- net /CLAMP: track 0.00 -> 46.2 mm
- net /X: track 0.00 -> 44.8 mm
- net /INTEN_B: track 0.00 -> 41.3 mm
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- added copper zone on B.Cu, net GND
Other:
- board outline added: 152.4 x 101.6 mm
- net class 250_or_hiz added: clearance 1.25, trace_width 0.25, via_dia 0.8, via_drill 0.4
- net class 400 added: clearance 2.5, trace_width 0.25, via_dia 0.8, via_drill 0.4

Commit message: Before second re-route
Parts:
- C28, C29: value 330n -> 220n
- C32: footprint Capacitor_THT:CP_Radial_D10.0mm_P2.50mm_P5.00mm -> Capacitor_THT:CP_Radial_D4.0mm_P1.50mm
- Q2, Q3: value ZTX558 -> MPSA92
- X1: value SLOPE -> S/DIV
- X11: value IB -> I-
- X6: value GO -> G+
- X7: value GI -> GW
- X8: value GG -> G-
- X9: value IT -> I+
- moved R14 56.7 mm to (157.5, 88.9), turned to -90 degrees
- moved R11 51.5 mm to (152.4, 101.6), turned to 90 degrees
- moved R9 50.7 mm to (137.2, 101.6), turned to 90 degrees
- moved XV1.4 48.3 mm to (160.0, 33.0)
- moved R13 41.2 mm to (158.8, 61.0)
- moved RV2 38.6 mm to (160.0, 78.7), turned to 180 degrees
- moved D22 38.6 mm to (131.4, 50.8), turned to 90 degrees
- moved R16 32.7 mm to (162.6, 44.5), turned to -90 degrees
- moved TP6 32.6 mm to (162.6, 110.5)
- moved TP1 30.1 mm to (160.0, 40.6)
- moved TP3 25.7 mm to (149.9, 40.6)
- moved TP2 25.7 mm to (144.8, 40.6)
- moved R8 25.6 mm to (132.1, 101.6)
- moved TP5 24.9 mm to (120.0, 86.4)
- moved R4 24.8 mm to (128.3, 111.8), turned to 90 degrees
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Connections:
- net Net-(NE1-Pad2) renamed /CRT Bias/NC250_5
- net Net-(Q2-Pad3) renamed /CRT Bias/NC250_2
- net Net-(Q3-Pad2) renamed /CRT Bias/NC250_3
- net Net-(Q3-Pad3) renamed /CRT Bias/NC400_3
- net Net-(R14-Pad1) renamed /CRT Bias/NC400_2
- net Net-(R16-Pad2) renamed /CRT Bias/NC250_1
- net Net-(R19-Pad1) renamed /CRT Bias/NC250_4
Routing:
- net GND: track 76.1 -> 0.00 mm, vias 0 -> 5
- net -400V: track 108.7 -> 37.4 mm, vias 1 -> 0
- net /SLOPE: track 37.3 -> 0.00 mm
- net +9V: track 415.4 -> 384.8 mm, vias 1 -> 0
- net /INTEN_B: track 41.3 -> 11.7 mm
- net Net-(D1-Pad1): track 32.4 -> 55.1 mm
- net Net-(Q9-Pad2): track 19.3 -> 40.5 mm
- net /INTEN_W: track 49.4 -> 28.8 mm, vias 0 -> 1
- net +400V: track 47.6 -> 66.3 mm
- net /K: track 87.5 -> 104.4 mm
- net /Sweep/~TRIG: track 30.7 -> 47.6 mm
- net /A2: track 21.1 -> 5.08 mm
- net Net-(D5-Pad2): track 6.35 -> 19.0 mm
- net /X: track 44.8 -> 32.6 mm, vias 0 -> 2
- net Net-(C39-Pad1): track 25.4 -> 37.3 mm
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Other:
- net class Default: via_dia 0.8 -> 1.4; via_drill 0.4 -> 0.6
- board text added: "+400V"
- board text added: "+9V"
- board text added: "-400V"
- board text added: "-9V"
- board text added: "<!> GRID BIAS"
- board text added: "A1"
- board text added: "A2"
- board text added: "ADJUST WITH CARE CCW FOR MINIMUM ADJUST AT MAX INTEN"
- board text added: "ASTIG"
- board text added: "DANGER! HIGH VOLTAGE in excess of ±400V with lethal current in all areas. Contact may KILL. System may retain charge."
- board text added: "F"
- board text added: "FOCUS"
- board text added: "G"
- board text added: "HOR GAIN"
- board text added: "HOR POS"
- board text added: "INTENSITY"
- board text added: "IN_GND"
- board text added: "IN_L"
- board text added: "IN_R"
- board text added: "K"
- board text added: "LEVEL"
- board text added: "Mini Audioscope © 2020 Alexis Lockwood. CC BY-NC-SA"
- board text added: "V/DIV"
- board text added: "VERT GAIN"
- board text added: "VERT POS"
- board text added: "X+"
- board text added: "X-"
- board text added: "Y+"
- board text added: "Y-"

Commit message: savesavesave
Parts:
- removed C37: 10n, Capacitor_THT:C_Disc_D4.7mm_W2.5mm_P5.00mm
- removed D21: 1N4148, Diode_THT:D_DO-35_SOD27_P7.62mm_Horizontal
- removed R23, R29, R49, R55: 470, Resistor_THT:R_Axial_DIN0207_L6.3mm_D2.5mm_P10.16mm_Horizontal
- removed R66, R70: 10k, Resistor_THT:R_Axial_DIN0207_L6.3mm_D2.5mm_P10.16mm_Horizontal
- removed R69: 4k7, Resistor_THT:R_Axial_DIN0207_L6.3mm_D2.5mm_P10.16mm_Horizontal
- removed R78: 100k, Resistor_THT:R_Axial_DIN0207_L6.3mm_D2.5mm_P10.16mm_Horizontal
- added C2: 33u/16, Capacitor_THT:CP_Radial_D4.0mm_P1.50mm, F.Cu at (91.4, 103.5)
- added C3: 33u/16, Capacitor_THT:CP_Radial_D4.0mm_P1.50mm, F.Cu at (95.2, 55.2)
- added C4: 33u/16, Capacitor_THT:CP_Radial_D4.0mm_P1.50mm, F.Cu at (115.6, 46.4)
- added C5: 33u/16, Capacitor_THT:CP_Radial_D4.0mm_P1.50mm, F.Cu at (94.0, 108.0)
- added C6: 22n, Capacitor_THT:C_Disc_D12.5mm_W5.0mm_P10.00mm, F.Cu at (71.8, 40.0)
- added C7: 22n, Capacitor_THT:C_Disc_D12.5mm_W5.0mm_P10.00mm, F.Cu at (152.4, 108.0)
- C38: footprint Capacitor_THT:C_Rect_L9.0mm_W5.1mm_P7.50mm_MKT -> Capacitor_THT:C_Rect_L13.0mm_W6.5mm_P7.50mm_P10.00mm
- Q18: value 2N3904 -> 2N7000
- moved R84 40.4 mm to (120.0, 72.4), turned to 90 degrees
- moved Q23 39.2 mm to (116.2, 80.0), turned to 90 degrees
- moved C38 30.9 mm to (109.9, 77.5)
- moved R34 30.4 mm to (72.4, 99.7), turned to 180 degrees
- moved D22 27.7 mm to (104.8, 58.4), turned to 0 degrees
- moved R91 26.2 mm to (102.2, 55.9), turned to 0 degrees
- moved C35 23.0 mm to (102.9, 40.0), turned to 180 degrees
- moved U8 19.2 mm to (95.2, 43.2)
- moved U6 18.5 mm to (94.0, 70.5)
- moved R89 17.6 mm to (78.1, 66.7)
- moved R83 17.1 mm to (105.4, 72.4), turned to 90 degrees
- moved C36 16.3 mm to (100.3, 65.4), turned to 180 degrees
- moved R30 15.6 mm to (45.1, 102.9), turned to -90 degrees
- moved R86 15.4 mm to (106.0, 43.2), turned to -90 degrees
- moved R73 15.3 mm to (87.6, 100.3)
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Connections:
- Q13 pad 1: Net-(Q13-Pad1) -> Net-(D19-Pad2)
- Q14 pad 1: Net-(Q14-Pad1) -> Net-(D20-Pad2)
- Q18 pad 2: Net-(Q18-Pad2) -> /Sweep/AUTO_TRIGGER
- Q6 pad 1: Net-(Q6-Pad1) -> Net-(D4-Pad2)
- Q7 pad 1: Net-(Q7-Pad1) -> Net-(D5-Pad2)
- R71 pad 1: Net-(R70-Pad2) -> Net-(R71-Pad1)
- RV9 pad 2: Net-(R70-Pad1) -> Net-(R71-Pad1)
- U4 pad 5: Net-(R66-Pad2) -> /GAIN_IN
- U5 pad 2: Net-(R69-Pad2) -> /OUT
- U5 pad 3: Net-(R70-Pad2) -> Net-(R71-Pad1)
Routing:
- net +9V: track 384.8 -> 447.8 mm
- net Net-(R71-Pad1): track 0.00 -> 24.2 mm
- net /SLOPE: track 0.00 -> 21.5 mm, vias 0 -> 2
- net Net-(Q22-Pad3): track 38.2 -> 17.0 mm, vias 1 -> 0
- net Net-(D1-Pad1): track 55.1 -> 36.8 mm
- net Net-(C38-Pad1): track 30.2 -> 14.5 mm
- net /OUT: track 75.5 -> 90.6 mm, vias 3 -> 5
- net /~BLANK: track 55.0 -> 40.5 mm
- net /Sweep/AUTO_TRIGGER: track 21.7 -> 7.25 mm
- net /Sweep/~TRIG: track 47.6 -> 33.2 mm
- net -9V: track 291.5 -> 305.7 mm, vias 4 -> 2
- net Net-(D20-Pad2): track 8.94 -> 22.8 mm
- net Net-(C39-Pad1): track 37.3 -> 23.8 mm
- net Net-(D4-Pad2): track 11.7 -> 23.3 mm
- net Net-(R86-Pad2): track 12.7 -> 22.5 mm, vias 0 -> 1
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
Commit message: Cleaned up
Parts:
- moved R48 1.27 mm to (66.7, 38.7)
- moved R52 1.27 mm to (59.1, 53.3)
- moved R53 1.27 mm to (62.9, 53.3)
- moved R65 1.27 mm to (43.8, 53.3)
- moved R66 1.27 mm to (51.4, 53.3)
- moved D5 0.64 mm to (61.6, 67.3)
- moved D6 0.64 mm to (65.4, 67.3)
- moved D7 0.64 mm to (47.0, 67.3)
- moved D8 0.64 mm to (50.2, 67.3)
- moved R60 0.64 mm to (55.9, 77.5)
- moved R43 0.63 mm to (55.2, 38.7)
- moved R56 0.63 mm to (40.0, 38.7)
- moved R61 0.63 mm to (47.6, 38.7)
- renumbered C2 to C1, C35 to C10, C36 to C11, C38 to C12, C39 to C13, C26 to C14, C1 to C15, C27 to C16, C28 to C17, C29 to C18, C30 to C19, C3 to C2, C31 to C20, C4 to C3, C5 to C4, C6 to C5, C7 to C6, C32 to C7, C33 to C8, C34 to C9, D22 to D1, D1 to D2, D2 to D3, D3 to D4, D19 to D5, D20 to D6, D4 to D7, D5 to D8, NE5 to NE1, NE1 to NE2, NE2 to NE3, Q17 to Q1, Q3 to Q10, Q4 to Q17, Q5 to Q18, Q6 to Q19, Q18 to Q2, Q7 to Q20, Q8 to Q21, Q9 to Q22, Q19 to Q3, Q20 to Q4, Q21 to Q5, Q22 to Q6, Q23 to Q7, Q1 to Q8, Q2 to Q9, R67 to R1, R79 to R10, R1 to R11, R80 to R12, R81 to R13, R82 to R14, R83 to R15, R84 to R16, R85 to R17, R86 to R18, R87 to R19, R68 to R2, R88 to R20, R89 to R21, R90 to R22, R91 to R23, R3 to R24, R4 to R25, R5 to R26, R6 to R27, R7 to R28, R8 to R29, R71 to R3, R9 to R30, R10 to R31, R11 to R32, R12 to R33, R13 to R34, R14 to R35, R15 to R36, R16 to R37, R17 to R38, R18 to R39, R72 to R4, R19 to R40, R46 to R41, R47 to R42, R48 to R43, R50 to R44, R51 to R45, R52 to R46, R53 to R47, R54 to R48, R56 to R49, R73 to R5, R59 to R50, R60 to R51, R57 to R52, R58 to R53, R20 to R54, R21 to R55, R22 to R56, R24 to R57, R25 to R58, R26 to R59, R74 to R6, R27 to R60, R28 to R61, R30 to R62, R33 to R63, R34 to R64, R31 to R65, R32 to R66, R61 to R67, R62 to R68, R64 to R69, R75 to R7, R65 to R70, R76 to R8, R77 to R9, RV9 to RV1, RV1 to RV2, RV2 to RV3, RV3 to RV4, RV7 to RV5, RV8 to RV6, RV4 to RV7, RV5 to RV8, U5 to U1, U6 to U2, U7 to U3, U8 to U4, U4 to U5
Routing:
- net /Horiz Defl/DEFL_INT+: track 15.0 -> 18.5 mm
- net +400V: track 73.2 -> 70.2 mm
- net Net-(D5-Pad2): track 24.6 -> 27.1 mm
- net /OUT: track 90.6 -> 88.4 mm
- net /DEFLX+: track 12.7 -> 10.7 mm
- net /Vert Defl/DEFL_INT+: track 8.83 -> 10.2 mm
- net Net-(D8-Pad2): track 28.6 -> 29.8 mm
- net /DEFLY-: track 9.68 -> 8.41 mm
- net /DEFLX-: track 10.7 -> 9.46 mm
- net /DEFLY+: track 9.15 -> 7.88 mm
- net /CLAMP: track 32.9 -> 32.0 mm
- net Net-(D7-Pad2): track 23.3 -> 24.2 mm
- net Net-(Q19-Pad2): track 17.1 -> 17.8 mm
- net Net-(D6-Pad2): track 22.8 -> 23.4 mm
- net /Horiz Defl/DEFL_INT-: track 12.4 -> 13.0 mm

Commit message: Version sent to fab
Parts:
- removed R35: 330k/HW, Resistor_THT:R_Axial_DIN0309_L9.0mm_D3.2mm_P12.70mm_Horizontal
- C5, C6: footprint Capacitor_THT:C_Disc_D12.5mm_W5.0mm_P10.00mm -> Capacitor_THT:C_Disc_D10.5mm_W5.0mm_P7.50mm
- Q12, Q15, Q18, Q21: value 2N4401 -> 2N3904
- R34: value 10k -> 180k
- RV1, RV2, RV5, RV6, RV7, RV8: footprint Potentiometer_THT:Potentiometer_Bourns_3339P_Vertical -> mini-audioscope:stock_pot
- RV3: value 1M -> 500k
- X1, X10, X11, X12, X13, X14, X15, X2, X3, X4, X5, X6, X7, X8, X9, XV1.10, XV1.11, XV1.2, XV1.3, XV1.4, XV1.6, XV1.7, XV1.8, XV1.9: footprint Connector_Pin:Pin_D0.7mm_L6.5mm_W1.8mm_FlatFork -> Connector_Pin:Pin_D1.1mm_L8.5mm_W2.5mm_FlatFork
- moved RV8 5.32 mm to (55.9, 102.6), turned to 0 degrees
- moved Q13 5.08 mm to (64.1, 57.8), turned to -90 degrees
- moved Q14 5.08 mm to (74.9, 57.8), turned to -90 degrees
- moved Q19 5.08 mm to (42.5, 57.8), turned to -90 degrees
- moved Q20 5.08 mm to (53.3, 57.8), turned to -90 degrees
- moved RV2 3.22 mm to (138.4, 111.1)
- moved X1 2.54 mm to (111.8, 119.4)
- moved X10 2.54 mm to (127.0, 119.4)
- moved X11 2.54 mm to (132.1, 119.4)
- moved X2 2.54 mm to (116.8, 119.4)
- moved X3 2.54 mm to (57.1, 119.4)
- moved X4 2.54 mm to (52.1, 119.4)
- moved X5 2.54 mm to (47.0, 119.4)
- moved X6 2.54 mm to (74.9, 119.4)
- moved X7 2.54 mm to (80.0, 119.4)
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Connections:
- Q13 pad 1: Net-(D5-Pad2) -> /Horiz Defl/DEFL_INT-
- Q13 pad 3: /Horiz Defl/DEFL_INT- -> Net-(D5-Pad2)
- Q14 pad 1: Net-(D6-Pad2) -> /Horiz Defl/DEFL_INT+
- Q14 pad 3: /Horiz Defl/DEFL_INT+ -> Net-(D6-Pad2)
- Q19 pad 1: Net-(D7-Pad2) -> /Vert Defl/DEFL_INT-
- Q19 pad 3: /Vert Defl/DEFL_INT- -> Net-(D7-Pad2)
- Q20 pad 1: Net-(D8-Pad2) -> /Vert Defl/DEFL_INT+
- Q20 pad 3: /Vert Defl/DEFL_INT+ -> Net-(D8-Pad2)
- R41 pad 1: +9V -> -9V
- R42 pad 2: -9V -> GND
- R54 pad 1: +9V -> -9V
- R55 pad 2: -9V -> GND
- RV3 pad 3: /CRT Bias/NC400_2 -> -400V
Routing:
- net -400V: track 42.5 -> 63.0 mm
- net -9V: track 305.7 -> 291.6 mm
- net Net-(Q18-Pad2): track 26.5 -> 39.3 mm
- net +9V: track 447.6 -> 438.4 mm
- net Net-(Q22-Pad2): track 40.8 -> 49.1 mm
- net Net-(Q13-Pad2): track 19.4 -> 27.2 mm
- net /CRT Bias/NC400_2: track 6.13 -> 0.00 mm
- net Net-(Q19-Pad2): track 17.8 -> 22.4 mm
- net Net-(R64-Pad2): track 11.8 -> 7.56 mm
- net Net-(C15-Pad2): track 49.5 -> 53.6 mm
- net /R: track 9.15 -> 6.61 mm
- net /L: track 9.15 -> 6.61 mm
- net /INTEN_W: track 24.4 -> 21.9 mm
- net /GAIN_IN: track 23.0 -> 20.5 mm
- net /SLOPE: track 21.5 -> 18.9 mm
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Other:
- net class 250_or_hiz: clearance 1.25 -> 1.27; trace_width 0.25 -> 0.508; via_dia 0.8 -> 0.8128; via_drill 0.4 -> 0.4064
- net class 400: clearance 2.5 -> 2.54; trace_width 0.25 -> 0.508; via_dia 0.8 -> 0.8128; via_drill 0.4 -> 0.4064
- net class Default: clearance 0.2 -> 0.2032; trace_width 0.25 -> 0.508; via_dia 1.4 -> 1.524; via_drill 0.6 -> 0.762
- rule trace_clearance: 0.2 -> 0.2032
- board text added: "A92"
- board text added: "ZTX"

Commit message: Schematic updates
Parts:
- C1, C2, C3, C4: value 33u/16 -> 33µ
- C11: value 47u -> 47µ
- C7: value 3u3 -> 3µ3
- R11: value 100k -> 10k
- R50, R51, R63, R64: value 10k -> 8k2
- RV6, RV8: value 2k5 -> 2k
